File: Prezenter/Prezenter.kicad_sch (KiCad schematic)
At the start: 26 parts, among them J1 TYPE-C-31-M-17, J2 Battery, J3 Laser, SW1 SW_Push_Dual, SW2 SW_Push_Dual, SW3 SW_Push_Dual, U1 DW01A, U2 FS8205A, U3 MCP73831-2-OT, U4 ESP32-WROOM-32

Commit message: Update
Parts:
- removed C1: 100nF, Capacitor_SMD:C_0805_2012Metric_Pad1.18x1.45mm_HandSolder, symbol Device:C
- removed C2, C4: 4.7uF, Capacitor_SMD:C_0805_2012Metric_Pad1.18x1.45mm_HandSolder, symbol Device:C
- removed C3: 10uF, Capacitor_SMD:C_0805_2012Metric_Pad1.18x1.45mm_HandSolder, symbol Device:C
- removed D1: RED, Capacitor_SMD:C_0805_2012Metric_Pad1.18x1.45mm_HandSolder, symbol Device:LED
- removed J1: TYPE-C-31-M-17, custom_library:USB_TYPE-C-31-M-17, symbol TYPE-C-31-M-17:TYPE-C-31-M-17
- removed R1: 1k, Resistor_SMD:R_0805_2012Metric_Pad1.20x1.40mm_HandSolder, symbol Device:R
- removed R2: 2k, Resistor_SMD:R_0805_2012Metric_Pad1.20x1.40mm_HandSolder, symbol Device:R
- removed R3: 100, Resistor_SMD:R_0805_2012Metric_Pad1.20x1.40mm_HandSolder, symbol Device:R
- removed R4: 470, Resistor_SMD:R_0805_2012Metric_Pad1.20x1.40mm_HandSolder, symbol Device:R
- removed S1: EG1218, digikey-footprints:Switch_Slide_11.6x4mm_EG1218, symbol dk_Slide-Switches:EG1218
- removed U1: DW01A, Package_TO_SOT_SMD:SOT-23-6, symbol dw01a:DW01A
- removed U2: FS8205A, Package_SO:TSSOP-8_4.4x3mm_P0.65mm, symbol fs8205a:FS8205A
- removed U3: MCP73831-2-OT, Package_TO_SOT_SMD:SOT-23-5, symbol Battery_Management:MCP73831-2-OT
- D1: renamed from D2; footprint Capacitor_SMD:C_0805_2012Metric_Pad1.18x1.45mm_HandSolder -> LED_THT:LED_D5.0mm
- J1: renamed from J2; value Battery -> Vin
- R1: renamed from R5; footprint Resistor_SMD:R_0805_2012Metric_Pad1.20x1.40mm_HandSolder -> Resistor_THT:R_Axial_DIN0207_L6.3mm_D2.5mm_P10.16mm_Horizontal
- R2: renamed from R6; footprint Resistor_SMD:R_0805_2012Metric_Pad1.20x1.40mm_HandSolder -> Resistor_THT:R_Axial_DIN0207_L6.3mm_D2.5mm_P10.16mm_Horizontal
- R3: renamed from R7; footprint Resistor_SMD:R_0805_2012Metric_Pad1.20x1.40mm_HandSolder -> Resistor_THT:R_Axial_DIN0207_L6.3mm_D2.5mm_P10.16mm_Horizontal
- R4: renamed from R8; footprint Resistor_SMD:R_0805_2012Metric_Pad1.20x1.40mm_HandSolder -> Resistor_THT:R_Axial_DIN0207_L6.3mm_D2.5mm_P10.16mm_Horizontal
- R5: renamed from R9; footprint Resistor_SMD:R_0805_2012Metric_Pad1.20x1.40mm_HandSolder -> Resistor_THT:R_Axial_DIN0207_L6.3mm_D2.5mm_P10.16mm_Horizontal
- renumbered J3 to J2, U4 to U1
Connections:
- net B- is gone; now on net GND: J1.1 (Pin_1)
- net VOUT is gone; now on net VCC: J1.2 (Pin_2)
- no-connect marks 45 -> 35
Other:
- note removed: "Charging Circuit"
- moved on the sheet: D1, J1, J2, R1, R2, R3, R4, R5, SW1, SW2, SW3, U1

Commit message: Update
Parts:
- added J2: Prog, Connector_PinHeader_2.54mm:PinHeader_1x04_P2.54mm_Vertical, symbol Connector:Conn_01x04_Pin
- renumbered J2 to J1, J1 to J3
Connections:
- net D0: now reaches U1.25 (IO0)
- net D0: now also J2.4 (Pin_4)
- net EN: now reaches U1.3 (EN)
- net EN: now also J2.3 (Pin_3)
- net RX: now reaches U1.34 (RXD0/IO3)
- net RX: now also J2.2 (Pin_2)
- net TX: now reaches U1.35 (TXD0/IO1)
- net TX: now also J2.1 (Pin_1)
- no-connect marks 35 -> 31
Other:
- moved on the sheet: J1, J3, SW1
