File: Prezenter/Prezenter.kicad_pcb (KiCad board)
At the start: 2 copper layers, 38.1 x 88.9 mm, 26 parts, among them J1 TYPE-C-31-M-17, J2 Battery, J3 Laser, SW1 SW_Push_Dual, SW2 SW_Push_Dual, SW3 SW_Push_Dual, U1 DW01A, U2 FS8205A, U3 MCP73831-2-OT, U4 ESP32-WROOM-32

Commit message: Update
Parts:
- removed C1: 100nF, Capacitor_SMD:C_0805_2012Metric_Pad1.18x1.45mm_HandSolder
- removed C2, C4: 4.7uF, Capacitor_SMD:C_0805_2012Metric_Pad1.18x1.45mm_HandSolder
- removed C3: 10uF, Capacitor_SMD:C_0805_2012Metric_Pad1.18x1.45mm_HandSolder
- removed D2: RED, Capacitor_SMD:C_0805_2012Metric_Pad1.18x1.45mm_HandSolder
- removed R6, R7: 100k, Resistor_SMD:R_0805_2012Metric_Pad1.20x1.40mm_HandSolder
- removed R8, R9: 10k, Resistor_SMD:R_0805_2012Metric_Pad1.20x1.40mm_HandSolder
- removed S1: EG1218, digikey-footprints:Switch_Slide_11.6x4mm_EG1218
- removed U2: FS8205A, Package_SO:TSSOP-8_4.4x3mm_P0.65mm
- removed U3: MCP73831-2-OT, Package_TO_SOT_SMD:SOT-23-5
- removed U4: ESP32-WROOM-32, RF_Module:ESP32-WROOM-32
- D1: footprint Capacitor_SMD:C_0805_2012Metric_Pad1.18x1.45mm_HandSolder -> LED_THT:LED_D5.0mm
- J1: value TYPE-C-31-M-17 -> Laser; footprint custom_library:USB_TYPE-C-31-M-17 -> Connector_PinHeader_2.54mm:PinHeader_1x02_P2.54mm_Vertical
- J2: value Battery -> Prog; footprint Connector_PinHeader_2.54mm:PinHeader_1x02_P2.54mm_Vertical -> Connector_PinHeader_2.54mm:PinHeader_1x04_P2.54mm_Vertical
- J3: value Laser -> Vin
- R1: value 1k -> 10k; footprint Resistor_SMD:R_0805_2012Metric_Pad1.20x1.40mm_HandSolder -> Resistor_THT:R_Axial_DIN0207_L6.3mm_D2.5mm_P10.16mm_Horizontal
- R2: value 2k -> 100k; footprint Resistor_SMD:R_0805_2012Metric_Pad1.20x1.40mm_HandSolder -> Resistor_THT:R_Axial_DIN0207_L6.3mm_D2.5mm_P10.16mm_Horizontal
- R3: value 100 -> 100k; footprint Resistor_SMD:R_0805_2012Metric_Pad1.20x1.40mm_HandSolder -> Resistor_THT:R_Axial_DIN0207_L6.3mm_D2.5mm_P10.16mm_Horizontal
- R4: value 470 -> 10k; footprint Resistor_SMD:R_0805_2012Metric_Pad1.20x1.40mm_HandSolder -> Resistor_THT:R_Axial_DIN0207_L6.3mm_D2.5mm_P10.16mm_Horizontal
- R5: footprint Resistor_SMD:R_0805_2012Metric_Pad1.20x1.40mm_HandSolder -> Resistor_THT:R_Axial_DIN0207_L6.3mm_D2.5mm_P10.16mm_Horizontal
- U1: value DW01A -> ESP32-WROOM-32; footprint Package_TO_SOT_SMD:SOT-23-6 -> RF_Module:ESP32-WROOM-32
- moved J1 77.2 mm to (182.2, 108.0), turned to 180 degrees
- moved J3 59.6 mm to (210.8, 163.8), turned to 0 degrees
- moved R4 52.4 mm to (186.7, 124.5)
- moved R3 46.3 mm to (213.4, 124.5)
- moved R2 46.3 mm to (208.3, 124.5)
- moved R1 44.2 mm to (201.9, 126.4), turned to 180 degrees
- moved U1 20.4 mm to (194.3, 157.1), turned to 90 degrees
- moved R5 7.43 mm to (181.6, 124.5)
- moved D1 2.67 mm to (210.8, 107.3)
- moved J2 2.27 mm to (210.8, 149.2), turned to 0 degrees
Connections:
- D1 pad 2: VUSB -> /D14
- J2 pad 1: B- -> /TX
- J2 pad 2: VOUT -> /RX
- J3 pad 2: Net-(J3-Pin_2) -> VCC
- R1 pad 1: Net-(U1-CS) -> /D26
- R2 pad 1: Net-(U3-PROG) -> /D35
- R2 pad 2: GND -> VCC
- R3 pad 1: Net-(U1-VCC) -> GND
- R3 pad 2: VOUT -> /D35
- R4 pad 1: Net-(U3-STAT) -> /D25
- R4 pad 2: Net-(D1-K) -> GND
- R5 pad 1: /D26 -> Net-(D1-K)
- SW1 pad 1: Net-(J3-Pin_2) -> Net-(J1-Pin_2)
- U1 pad 1: Net-(U1-OD) -> GND
- U1 pad 2: Net-(U1-CS) -> VCC
- U1 pad 3: Net-(U1-OC) -> /EN
- U1 pad 5: Net-(U1-VCC) -> unconnected-(U1-SENSOR_VN-Pad5)
- U1 pad 6: B- -> unconnected-(U1-IO34-Pad6)
Other:
- board size 38.1 x 88.9 mm -> 38.1 x 69.8 mm

Commit message: Update
Routing:
- net VCC: track 0.00 -> 126.1 mm
- net /D26: track 0.00 -> 65.8 mm, vias 0 -> 1
- net /D14: track 0.00 -> 65.0 mm, vias 0 -> 1
- net /D35: track 0.00 -> 64.1 mm, vias 0 -> 1
- net /D25: track 0.00 -> 52.4 mm, vias 0 -> 1
- net Net-(D1-K): track 0.00 -> 37.8 mm
- net /EN: track 0.00 -> 36.0 mm
- net /TX: track 0.00 -> 23.7 mm
- net /RX: track 0.00 -> 23.0 mm
- net /D0: track 0.00 -> 13.3 mm
- net Net-(J1-Pin_2): track 0.00 -> 11.5 mm
- added copper zone on B.Cu, net GND
- added copper zone on F.Cu, net GND
Other:
- board text added: "v1"
